File: Electrical/Segway/Segway.kicad_sch (KiCad schematic)
At the start: 11 parts

Commit message: big electrcal changes, rev 2 electronics settled
Parts:
- removed A?: Arduino_UNO_R3, Module:Arduino_UNO_R3, symbol MCU_Module:Arduino_UNO_R3
- removed C? (x2): CAP, symbol pspice:CAP
- removed D?: DIODE, symbol pspice:DIODE
- removed M? (x2): Motor_DC, symbol Motor:Motor_DC
- removed SW?: SW_SPST, symbol Switch:SW_SPST
- removed U?: L7805, symbol Regulator_Linear:L7805
- added U? (x2): BOB-12009, BOB-12009:CONV_BOB-12009, symbol IIC_Logic_Shifter:BOB-12009
- added U? (x2): GearMotor, symbol IIC_Logic_Shifter:GearMotor
- added U?: Raspberry Pi Pico, SC0915:MODULE_SC0915, symbol Raspberry_Pi_Pico:SC0915
- added U?: BuckConverter, symbol IIC_Logic_Shifter:BuckConverter
- added U? (x3): HC-SR04, HC-SR04:XCVR_HC-SR04, symbol HC-SR04:HC-SR04
- added U?: NRF24L01_Breakout, RF_Module:nRF24L01_Breakout, symbol RF:NRF24L01_Breakout
Connections:
- net VDC: now reaches U?.9 (Vss)
- net VDC: now also BT?.1 (+), U?. (Out-)
- net +3V3: now reaches U?.13 (VDD)
- net +3V3: now also U?.11 (EnB), U?.4 (Vs), U?.6 (EnA), U?. (Encoder+), U?. (Encoder+), U?.2 (VCC), U?.36 (3V3_OUT), U?.LV, U?.LV
- net at U?.12 (IN4): now also U?.34 (GP28)
- net at U?.10 (IN3): now also U?.32 (GP27)
- net at U?.7 (IN2): now also U?.31 (GP26)
- net at U?.5 (IN1): now also U?.29 (GP22)
- net at U?.24 (SDA): now also U?.1 (GP0)
- net at U?.23 (SCL): now also U?.2 (GP1)
- net GND: now reaches U?.18 (GND)
- net GND: now also BT?.2 (-), U?. (Out-), U?.1 (GND), U?.2 (Encoder-), U?.2 (Encoder-), U?.4 (GND), U?.4 (GND), U?.4 (GND), U?.GND_1 (GND), U?.GND_2 (GND)
- net at U?.13 (OUT3): now also U?.1 (Motor+)
- net at U?.14 (OUT4): now also U?.6 (Motor-)
- net at U?.2 (OUT1): now also U?.1 (Motor+)
- net at U?.3 (OUT2): now also U?.6 (Motor-)
- new net: U?.2 (TRIG), U?.HV1 (x2)
- new net: U?.3 (ECHO), U?.HV2 (x2)
- new net: U?.26 (GP20), U?.LV1
- new net: U?.27 (GP21), U?.LV2
- new net: U?.13 (GND), U?.18 (GND), U?.23 (GND), U?.28 (GND), U?.3 (GND), U?.38 (GND), U?.8 (GND), U?.D2 (GND)
- new net: U?.21 (GP16), U?.LV1
- new net: U?.22 (GP17), U?.LV2
- new net: U?.24 (GP18), U?.LV3
- new net: U?.25 (GP19), U?.LV4
- new net: U?.6 (MOSI), U?.7 (GP5)
- new net: U?.7 (MISO), U?.9 (GP6)
- new net: U?.A (USB_SHIELD), U?.B (USB_SHIELD), U?.C (USB_SHIELD), U?.D (USB_SHIELD)
- new net: U?.GND_1 (GND), U?.GND_2 (GND)
- new net: U?.2 (TRIG), U?.HV3
- new net: U?.3 (ECHO), U?.HV4
- new net +5V: U?. (Out-), U?.1 (VCC), U?.1 (VCC), U?.1 (VCC), U?.40 (VBUS), U?.HV, U?.HV
Other:
- title: Balancing Electronics -> Segway Robot
- moved on the sheet: BT?, U?

Commit message: regrouping, move to micropython
Connections:
- net GND: now also U?.13 (GND), U?.18 (GND), U?.23 (GND), U?.28 (GND), U?.3 (GND), U?.38 (GND), U?.8 (GND), U?.8 (GND), U?.D2 (GND)
- net at U?.3 (EncoderA): now also U?.16 (GP12)
- net at U?.4 (EncoderB): now also U?.15 (GP11)
- net at U?.10 (GP7): now also U?.3 (CE)
- net at U?.11 (GP8): now also U?.4 (~{CSN})
- net at U?.12 (GP9): now also U?.4 (EncoderB)
- net at U?.14 (GP10): now also U?.3 (EncoderA)
Changed lines of the file:
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@@
   (title_block
     (title "Segway Robot")
-    (date "2023-09-03")
-    (rev "0")
+    (date "2023-11-28")
+    (rev "2.1")
     (company "Senior Design")
     (comment 1 "FOR REFERENCE ONLY")
@@
   (junction (at 226.06 48.26) (diameter 0) (color 0 0 0 0)
   )
+  (junction (at 191.77 132.08) (diameter 0) (color 0 0 0 0)
+  )
   (junction (at 210.82 66.04) (diameter 0) (color 0 0 0 0)
   )
@@
     (stroke (width 0) (type default) (color 0 0 0 0))
   )
+  (wire (pts (xy 227.33 104.14) (xy 227.33 144.78))
+    (stroke (width 0) (type default) (color 0 0 0 0))
+  )
   (wire (pts (xy 175.26 71.12) (xy 170.18 71.12))
     (stroke (width 0) (type default) (color 0 0 0 0))
   )
+  (wire (pts (xy 236.22 124.46) (xy 231.14 124.46))
+    (stroke (width 0) (type default) (color 0 0 0 0))
+  )
   (wire (pts (xy 160.02 38.1) (xy 160.02 57.15))
     (stroke (width 0) (type default) (color 0 0 0 0))
   )
+  (wire (pts (xy 106.68 105.41) (xy 109.22 105.41))
+    (stroke (width 0) (type default) (color 0 0 0 0))
+  )
   (wire (pts (xy 186.69 132.08) (xy 186.69 133.35))
     (stroke (width 0) (type default) (color 0 0 0 0))
@@
     (stroke (width 0) (type default) (color 0 0 0 0))
   )
+  (wire (pts (xy 93.98 97.79) (xy 109.22 97.79))
+    (stroke (width 0) (type default) (color 0 0 0 0))
+  )
   (wire (pts (xy 219.71 43.18) (xy 219.71 45.72))
     (stroke (width 0) (type default) (color 0 0 0 0))
@@
     (stroke (width 0) (type default) (color 0 0 0 0))
   )
+  (wire (pts (xy 105.41 102.87) (xy 109.22 102.87))
+    (stroke (width 0) (type default) (color 0 0 0 0))
+  )
   (wire (pts (xy 187.96 96.52) (xy 191.77 96.52))
     (stroke (width 0) (type default) (color 0 0 0 0))
@@
     (stroke (width 0) (type default) (color 0 0 0 0))
   )
+  (wire (pts (xy 77.47 106.68) (xy 91.44 106.68))
+    (stroke (width 0) (type default) (color 0 0 0 0))
+  )
   (wire (pts (xy 78.74 77.47) (xy 109.22 77.47))
     (stroke (width 0) (type default) (color 0 0 0 0))
@@
     (stroke (width 0) (type default) (color 0 0 0 0))
   )
+  (wire (pts (xy 107.95 144.78) (xy 107.95 107.95))
+    (stroke (width 0) (type default) (color 0 0 0 0))
+  )
   (wire (pts (xy 213.36 99.06) (xy 236.22 99.06))
     (stroke (width 0) (type default) (color 0 0 0 0))
@@
     (stroke (width 0) (type default) (color 0 0 0 0))
   )
+  (wire (pts (xy 229.87 147.32) (xy 105.41 147.32))
+    (stroke (width 0) (type default) (color 0 0 0 0))
+  )
   (wire (pts (xy 88.9 116.84) (xy 88.9 92.71))
     (stroke (width 0) (type default) (color 0 0 0 0))
@@
     (stroke (width 0) (type default) (color 0 0 0 0))
   )
+  (wire (pts (xy 91.44 106.68) (xy 91.44 95.25))
+    (stroke (width 0) (type default) (color 0 0 0 0))
+  )
   (wire (pts (xy 175.26 106.68) (xy 175.26 116.84))
     (stroke (width 0) (type default) (color 0 0 0 0))
@@
     (stroke (width 0) (type default) (color 0 0 0 0))
   )
+  (wire (pts (xy 236.22 106.68) (xy 228.6 106.68))
+    (stroke (width 0) (type default) (color 0 0 0 0))
+  )
+  (wire (pts (xy 106.68 146.05) (xy 106.68 105.41))
+    (stroke (width 0) (type default) (color 0 0 0 0))
+  )
   (wire (pts (xy 163.83 111.76) (xy 163.83 105.41))
     (stroke (width 0) (type default) (color 0 0 0 0))
@@
     (stroke (width 0) (type default) (color 0 0 0 0))
   )
+  (wire (pts (xy 104.14 100.33) (xy 109.22 100.33))
+    (stroke (width 0) (type default) (color 0 0 0 0))
+  )
   (wire (pts (xy 210.82 35.56) (xy 214.63 35.56))
     (stroke (width 0) (type default) (color 0 0 0 0))
@@
     (stroke (width 0) (type default) (color 0 0 0 0))
   )
+  (wire (pts (xy 228.6 106.68) (xy 228.6 146.05))
+    (stroke (width 0) (type default) (color 0 0 0 0))
+  )
+  (wire (pts (xy 231.14 124.46) (xy 231.14 148.59))
+    (stroke (width 0) (type default) (color 0 0 0 0))
+  )
   (wire (pts (xy 222.25 45.72) (xy 222.25 48.26))
     (stroke (width 0) (type default) (color 0 0 0 0))
@@
     (stroke (width 0) (type default) (color 0 0 0 0))
   )
+  (wire (pts (xy 228.6 146.05) (xy 106.68 146.05))
+    (stroke (width 0) (type default) (color 0 0 0 0))
+  )
   (wire (pts (xy 171.45 73.66) (xy 171.45 97.79))
     (stroke (width 0) (type default) (color 0 0 0 0))
   )
+  (wire (pts (xy 91.44 95.25) (xy 109.22 95.25))
+    (stroke (width 0) (type default) (color 0 0 0 0))
+  )
   (wire (pts (xy 210.82 31.75) (xy 210.82 35.56))
     (stroke (width 0) (type default) (color 0 0 0 0))
@@
     (stroke (width 0) (type default) (color 0 0 0 0))
   )
+  (wire (pts (xy 227.33 144.78) (xy 107.95 144.78))
+    (stroke (width 0) (type default) (color 0 0 0 0))
+  )
   (wire (pts (xy 228.6 31.75) (xy 218.44 31.75))
     (stroke (width 0) (type default) (color 0 0 0 0))
@@
     (stroke (width 0) (type default) (color 0 0 0 0))
   )
+  (wire (pts (xy 231.14 148.59) (xy 104.14 148.59))
+    (stroke (width 0) (type default) (color 0 0 0 0))
+  )
+  (wire (pts (xy 191.77 132.08) (xy 191.77 133.35))
+    (stroke (width 0) (type default) (color 0 0 0 0))
+  )
   (wire (pts (xy 165.1 85.09) (xy 160.02 85.09))
     (stroke (width 0) (type default) (color 0 0 0 0))
@@
     (stroke (width 0) (type default) (color 0 0 0 0))
   )
+  (wire (pts (xy 229.87 121.92) (xy 229.87 147.32))
+    (stroke (width 0) (type default) (color 0 0 0 0))
+  )
   (wire (pts (xy 168.91 48.26) (xy 168.91 92.71))
     (stroke (width 0) (type default) (color 0 0 0 0))
@@
     (stroke (width 0) (type default) (color 0 0 0 0))
   )
+  (wire (pts (xy 236.22 121.92) (xy 229.87 121.92))
+    (stroke (width 0) (type default) (color 0 0 0 0))
+  )
   (wire (pts (xy 29.21 48.26) (xy 53.34 48.26))
     (stroke (width 0) (type default) (color 0 0 0 0))
@@
     (stroke (width 0) (type default) (color 0 0 0 0))
   )
+  (wire (pts (xy 160.02 138.43) (xy 162.56 138.43))
+    (stroke (width 0) (type default) (color 0 0 0 0))
+  )
   (wire (pts (xy 217.17 40.64) (xy 210.82 40.64))
     (stroke (width 0) (type default) (color 0 0 0 0))
@@
     (stroke (width 0) (type default) (color 0 0 0 0))
   )
+  (wire (pts (xy 236.22 104.14) (xy 227.33 104.14))
+    (stroke (width 0) (type default) (color 0 0 0 0))
+  )
   (wire (pts (xy 167.64 45.72) (xy 167.64 90.17))
     (stroke (width 0) (type default) (color 0 0 0 0))
   )
+  (wire (pts (xy 93.98 111.76) (xy 93.98 97.79))
+    (stroke (width 0) (type default) (color 0 0 0 0))
+  )
   (wire (pts (xy 226.06 83.82) (xy 226.06 87.63))
     (stroke (width 0) (type default) (color 0 0 0 0))
@@
     (stroke (width 0) (type default) (color 0 0 0 0))
   )
+  (wire (pts (xy 105.41 147.32) (xy 105.41 102.87))
+    (stroke (width 0) (type default) (color 0 0 0 0))
+  )
   (wire (pts (xy 82.55 80.01) (xy 109.22 80.01))
     (stroke (width 0) (type default) (color 0 0 0 0))
@@
     (stroke (width 0) (type default) (color 0 0 0 0))
   )
+  (wire (pts (xy 77.47 111.76) (xy 93.98 111.76))
+    (stroke (width 0) (type default) (color 0 0 0 0))
+  )
   (wire (pts (xy 218.44 31.75) (xy 218.44 43.18))
     (stroke (width 0) (type default) (color 0 0 0 0))
   )
+  (wire (pts (xy 107.95 107.95) (xy 109.22 107.95))
+    (stroke (width 0) (type default) (color 0 0 0 0))
+  )
   (wire (pts (xy 233.68 119.38) (xy 236.22 119.38))
     (stroke (width 0) (type default) (color 0 0 0 0))
@@
   (wire (pts (xy 175.26 62.23) (xy 175.26 66.04))
     (stroke (width 0) (type default) (color 0 0 0 0))
+  )
+  (wire (pts (xy 104.14 148.59) (xy 104.14 100.33))
+    (stroke (width 0) (type default) (color 0 0 0 0))
+  )
+  (symbol (lib_id "power:GND") (at 162.56 138.43 0) (unit 1)
+    (in_bom yes) (on_board yes) (fields_autoplaced)
+    (property "Reference" "#PWR?" (id 0) (at 162.56 144.78 0)
+      (effects (font (size 1.27 1.27)) hide)
+    )
+    (property "Value" "GND" (id 1) (at 162.56 143.51 0))
+    (property "Footprint" "" (id 2) (at 162.56 138.43 0)
+      (effects (font (size 1.27 1.27)) hide)
+    )
+    (property "Datasheet" "" (id 3) (at 162.56 138.43 0)
+      (effects (font (size 1.27 1.27)) hide)
+    )
+    (pin "1")
+  )
+  (symbol (lib_id "power:GND") (at 191.77 133.35 0) (unit 1)
+    (in_bom yes) (on_board yes) (fields_autoplaced)
+    (property "Reference" "#PWR?" (id 0) (at 191.77 139.7 0)
+      (effects (font (size 1.27 1.27)) hide)
+    )
+    (property "Value" "GND" (id 1) (at 191.77 138.43 0))
+    (property "Footprint" "" (id 2) (at 191.77 133.35 0)
+      (effects (font (size 1.27 1.27)) hide)
+    )
+    (property "Datasheet" "" (id 3) (at 191.77 133.35 0)
+      (effects (font (size 1.27 1.27)) hide)
+    )
+    (pin "1")
   )
   (symbol (lib_id "power:GND") (at 233.68 134.62 0) (unit 1)
@@
   )
   (symbol_instances
+    (path "/0078d5b0-3e2b-404e-a167-d259131e3725"
+      (reference "#PWR?") (unit 1) (value "GND") (footprint "")
+    )
+    (path "/0b63576e-20ab-4f8c-943c-b8c5b7bf46f2"
+      (reference "#PWR?") (unit 1) (value "GND") (footprint "")
+    )
     (path "/0c716547-4adb-4d8d-9afd-d21165d0dbbb"
       (reference "#PWR?") (unit 1) (value "GND") (footprint "")
